File: hardware/EV1/EV1.kicad_sch (KiCad schematic)
At the start: 37 parts, among them J1 Conn_01x04_Male, J2 Conn_01x04_Male, J3 Conn_01x09_Male, J4 Conn_01x07_Male, J5 Conn_01x08_Male, J6 Conn_01x04_Male, J7 Conn_01x06_Male, P1 USB_C_Plug, SW1 SW_SPDT, SW2 SW_Push, U1 STM32F405RGTx, U2 AMS1117-3.3, Y1 25mhz

Commit message: EV1 updated
Parts:
- removed C3: 10p, Capacitor_SMD:C_0805_2012Metric, symbol Device:C
- removed J6: Conn_01x04_Male, Connector_JST:JST_EH_S4B-EH_1x04_P2.50mm_Horizontal, symbol Connector:Conn_01x04_Male
- removed SW1: SW_SPDT, Button_Switch_SMD:SW_SPDT_PCM12, symbol Switch:SW_SPDT
- removed Y1: 25mhz, Oscillator:Oscillator_SMD_SeikoEpson_SG8002LB-4Pin_5.0x3.2mm, symbol Device:Crystal_GND24
- added C5: 100n, Capacitor_SMD:C_0805_2012Metric, symbol Device:C
- added J6, J8: Conn_01x06_Male, Connector_JST:JST_EH_S6B-EH_1x06_P2.50mm_Horizontal, symbol Connector:Conn_01x06_Male
- added R11, R12: 5k1, Resistor_SMD:R_0805_2012Metric, symbol Device:R
- added R13: 4k7, Resistor_SMD:R_0805_2012Metric, symbol Device:R
- added SW1: SW_Push, Button_Switch_SMD:SW_DIP_SPSTx01_Slide_6.7x4.1mm_W6.73mm_P2.54mm_LowProfile_JPin, symbol Switch:SW_Push
- added X1: SG-5032CAN, Oscillator:Oscillator_SMD_SeikoEpson_SG8002LB-4Pin_5.0x3.2mm, symbol Oscillator:SG-5032CAN
- C4: value 10p -> 100n
- R1: value 1k5 -> 150
- R2: value 10k -> 4k7
Connections:
- net SW_BOOT0 is gone; now on net RESET: R2.1
- net +3.3V: now also C4.1, R2.2, J6.1 (Pin_1), J8.1 (Pin_1), SW1.1, X1.4 (VCC); no longer SW2.2
- net BOOT0: now also R13.2, SW1.2; no longer R2.2
- net GND: now also SW2.1, C5.1, J6.5 (Pin_5), J6.6 (Pin_6), J8.5 (Pin_5), J8.6 (Pin_6), R11.1, R12.1, R13.1, X1.2 (GND)
- net HSE_IN: now also X1.3 (OUT)
- net USART2_RX: now also J8.3 (Pin_3)
- net USART2_TX: now also J8.4 (Pin_4)
- net VBUS: now also J8.2 (Pin_2); no longer D2.2 (A), U2.3 (VI)
- net RESET: now reaches U1.7 (NRST)
- net RESET: now also SW2.2, C5.2, J6.4 (Pin_4); no longer SW2.1
- net SWD_DIO: now reaches U1.46 (PA13)
- net SWD_DIO: now also J6.3 (Pin_3)
- net SWD_CLK: now reaches U1.49 (PA14)
- net SWD_CLK: now also J6.2 (Pin_2)
- net at P1.A5 (CC): now also R12.2
- net at P1.B5 (VCONN): now also R11.2
- net HSE_OUT: no longer names the net of U1.6 (PH1)
- net HSE_OUT: no longer C4.1
- new net: D2.2 (A), U2.3 (VI)
- no-connect marks 37 -> 35
Other:
- note added: "BOOT Button"
- note added: "STLink Connector"
- note removed: "BOOT Slide"
- note removed: "V_IN"
- moved on the sheet: C11, C12, C13, C14, C4, D2, J2, J3, J5, SW2

Commit message: Finished Version of EV1
Parts:
- removed J1, J2: Conn_01x04_Male, Connector_JST:JST_EH_S4B-EH_1x04_P2.50mm_Horizontal, symbol Connector:Conn_01x04_Male
- removed J3: Conn_01x09_Male, Connector_JST:JST_XH_S9B-XH-A-1_1x09_P2.50mm_Horizontal, symbol Connector:Conn_01x09_Male
- removed J4: Conn_01x07_Male, Connector_JST:JST_XH_S7B-XH-A_1x07_P2.50mm_Horizontal, symbol Connector:Conn_01x07_Male
- removed J5: Conn_01x08_Male, Connector_JST:JST_XH_S8B-XH-A-1_1x08_P2.50mm_Horizontal, symbol Connector:Conn_01x08_Male
- removed J6, J7, J8: Conn_01x06_Male, Connector_JST:JST_EH_S6B-EH_1x06_P2.50mm_Horizontal, symbol Connector:Conn_01x06_Male
- removed P1: USB_C_Plug, Connector_USB:USB_C_Plug_Molex_105444, symbol Connector:USB_C_Plug
- added J9: USB_C_Receptacle, Connector_USB:USB_C_Receptacle_HRO_TYPE-C-31-M-12, symbol Connector:USB_C_Receptacle
- added U10, U5, U8: 1x6_connector, 1x4 pin download:1x6_connector, symbol connector_library:1x6_connector
- added U3: 1x8_connector, 1x4 pin download:1X8_CONNECTOR, symbol connector_library:1x8_connector
- added U4, U9: 1x4_connector, 1x4 pin download:1x4_connector, symbol connector_library:1x4_connector
- added U6: 1x7_connector, 1x4 pin download:1x7_connector, symbol connector_library:1x7_connector
- added U7: 1x9_connector, 1x4 pin download:1x9_connector, symbol connector_library:1x9_connector
- 120R1: footprint Inductor_SMD:L_0805_2012Metric -> Connector_USB:USB_C_Receptacle_HRO_TYPE-C-31-M-12
Connections:
- net +3.3V: now also U10.6, U3.1, U4.4, U5.6, U6.1, U7.1, U8.6, U9.4
- net BB_COLS_2: now also U6.2
- net BB_COLS_3: now also U6.3
- net BB_COLS_4: now also U6.4
- net BB_COLS_5: now also U6.5
- net BB_COLS_6: now also U6.6
- net BB_ROW_2: now also U7.2
- net BB_ROW_3: now also U7.3
- net BB_ROW_4: now also U7.4
- net BB_ROW_5: now also U7.5
- net BB_ROW_6: now also U7.6
- net BB_ROW_7: now also U7.7
- net BB_ROW_8: now also U7.8
- net BL_PA4: now also U3.3
- net CS_PA1: now also U3.4
- net DC_PB0: now also U3.5
- net GND: now also J9.A1 (GND), J9.A12 (GND), J9.B1 (GND), J9.B12 (GND), U10.1, U10.2, U3.8, U4.1, U5.1, U5.2, U6.7, U7.9, U8.1, U9.1
- net I2C_SCL: now also U4.2
- net I2C_SDA: now also U4.3
- net IO_PC6: now also U8.2
- net IO_PC7: now also U8.3
- net IO_PC8: now also U8.4
- net IO_PC9: now also U8.5
- net MOSI_SPI: now also U3.6
- net RESET: now also U5.3
- net RST_PA6: now also U3.2
- net SCK_SPI: now also U3.7
- net SWD_CLK: now also U5.5
- net SWD_DIO: now also U5.4
- net USART2_RX: now also U10.4
- net USART2_TX: now also U10.3
- net USART_3_RX: now also U9.3
- net USART_3_TX: now also U9.2
- net VBUS: now also J9.A4 (VBUS), J9.A9 (VBUS), J9.B4 (VBUS), J9.B9 (VBUS), U10.5
- net at R11.2: now also J9.B5 (CC2)
- net at R10.2: now also J9.A7 (D-), J9.B7 (D-)
- net at R9.2: now also J9.A6 (D+), J9.B6 (D+)
- net at R12.2: now also J9.A5 (CC1)
Other:
- note added: "U4-J1 U5-J6 U6-J4 U7-J3 U8-J7 U9-J2 U10-J8 U3-J5"
- title: EV1 Initial Design -> Finn Berg - EV1
- moved on the sheet: D2, R10, R11, R12, R9

Commit message: EV3 Final Board and Schematic
Parts:
- added CR?: M24C02-RDW6TP, ESP32-S3-WROOM-1-N8R2:M24C02-RDW6TP, symbol m24c02-rdw6tp:M24C02-RDW6TP
- added U?: ESP32-S3-WROOM-1-N8R2, ESP32-S3-WROOM-1-N8R2:ESP32-S3-WROOM-1-N8R2, symbol ESP32-S3-WROOM-1-N8R2:ESP32-S3-WROOM-1-N8R2
- added U?: WM8960CGEFL/RV, ESP32-S3-WROOM-1-N8R2:QFN50P500X500X90-33N, symbol Audio Interface:WM8960CGEFL/RV
- added U? (x2): 74HC4066D, ESP32-S3-WROOM-1-N8R2:SOIC127P600X175-14N, symbol 74HC4066D:74HC4066D
- added U?: CH340N, CH340C:SOIC127P600X180-16N, symbol CH340N:CH340N
- 120R1: footprint Connector_USB:USB_C_Receptacle_HRO_TYPE-C-31-M-12 -> Inductor_SMD:L_0805_2012Metric
Connections:
- new net: U?.1 (GND), U?.40 (GND), U?.41_1 (GND), U?.41_2 (GND), U?.41_3 (GND), U?.41_4 (GND), U?.41_5 (GND), U?.41_6 (GND), U?.41_7 (GND), U?.41_8 (GND), U?.41_9 (GND)
Other:
- note added: "-Add test points to key signals -Add 0ohm resistors to key traces -Add ESP32-S3-WROOM-1-N8R2 -Add heat sink to power -Add CH340N for USB serial -Add M24C02-RMN6TP eeprom -Add two 74HC4066 serial switches -Add WM8960 for audio testing -Add keyboard connector"
- note removed: "Next Steps: -Connect any remaining pieces: (LED's, Potentiometer, Second crystal?) -Assign footprints and JCLPCB part ID -Make headers for rest of IO pins -Show Brett to see if issues -Show Cullen to see if issues -Check requirements for PCB at JCLPCB -Begin PCB Design"
- note removed: "Parts Left: -Second crystal oscilator -C5 and C6? -Any remaining LED's -AMS1117"
- note removed: "U4-J1 U5-J6 U6-J4 U7-J3 U8-J7 U9-J2 U10-J8 U3-J5"
- moved on the sheet: 120R1, C1, C10, C11, C12, C13, C14, C2, C4, C5, C8, C9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
