File: hardware/EV2/EV2 Final Board.kicad_sch (KiCad schematic)
At the start: 87 parts, among them J9 USB_C_Receptacle, SW1 SW_Push, SW2 SW_Push, SW3 SW_Push, SW4 SW_Push, SW5 SW_DIP_x02, SW6 SW_DIP_x02, SW7 SW_DIP_x02, SW8 SW_DIP_x02, U1 STM32F405RGTx, U11 ESP32-S3-WROOM-1-N8R2, U14 WM8960CGEFL/RV, U15 CH340N, U16 BM20B(0.8)-24DS-0.4V(51), U17 1x4_connector, U18 1x6_connector, U19 1x6_connector, U2 AMS1117-3.3, U20 1x8_connector, U3 1x8_connector, U4 USBLC6-2P6, U5 1x6_connector, U6 1x7_connector, U7 1x9_connector, U8 1x6_connector, U9 1x4_connector, X1 SG-5032CAN

Commit message: EV2 Final Board Design
Parts:
- removed R21, R22: 560, Resistor_SMD:R_0805_2012Metric, symbol Device:R
- removed SW5, SW6, SW7, SW8: SW_DIP_x02, Button_Switch_SMD:SW_DIP_SPSTx02_Slide_6.7x6.64mm_W6.73mm_P2.54mm_LowProfile_JPin, symbol Switch:SW_DIP_x02
- CR1: footprint ESP32-S3-WROOM-1-N8R2:M24C02-RDW6TP -> ESP32-S3-WROOM-1-N8R2:New_ESP32_M24C02-RMN6TP
Connections:
- net UART2_RX is gone; now on net ESP_UART1_TX: U1.17 (PA3)
- net UART2_TX is gone; now on net ESP_UART1_RX: U1.16 (PA2)
- net +3.3V: no longer U3.1
- net UART1_RX: now also R9.1
- net UART1_TX: now also R10.1
- net VBUS: now also D2.2 (A), U3.1; no longer D2.1 (K)
- net at U2.3 (VI): now also D2.1 (K); no longer D2.2 (A)
Other:
- moved on the sheet: D2
