File: hardware/EV2/EV2 final Board.kicad_pcb (KiCad board)
At the start: 2 copper layers, 129.6 x 73.1 mm, 87 parts, among them J9 USB_C_Receptacle, SW1 SW_Push, SW2 SW_Push, SW3 SW_Push, SW4 SW_Push, SW5 SW_DIP_x02, SW6 SW_DIP_x02, SW7 SW_DIP_x02, SW8 SW_DIP_x02, U1 STM32F405RGTx, U11 ESP32-S3-WROOM-1-N8R2, U14 WM8960CGEFL/RV, U15 CH340N, U16 BM20B(0.8)-24DS-0.4V(51), U17 1x4_connector, U18 1x6_connector, U19 1x6_connector, U2 AMS1117-3.3, U20 1x8_connector, U3 1x8_connector, U4 USBLC6-2P6, U5 1x6_connector, U6 1x7_connector, U7 1x9_connector, U8 1x6_connector, U9 1x4_connector, X1 SG-5032CAN

Commit message: EV2 Final Board Design
Parts:
- removed R21, R22: 560, Resistor_SMD:R_0805_2012Metric
- removed SW5, SW6, SW7, SW8: SW_DIP_x02, Button_Switch_SMD:SW_DIP_SPSTx02_Slide_6.7x6.64mm_W6.73mm_P2.54mm_LowProfile_JPin
- CR1: footprint ESP32-S3-WROOM-1-N8R2:M24C02-RDW6TP -> ESP32-S3-WROOM-1-N8R2:New_ESP32_M24C02-RMN6TP
- moved CR1 28.4 mm to (122.6, 48.3)
- turned D2 to 180 degrees
Connections:
- D2 pad 1: VBUS -> Net-(D2-Pad1)
- D2 pad 2: Net-(D2-Pad2) -> VBUS
- R10 pad 1: Net-(R10-Pad1) -> /UART1_TX
- R9 pad 1: Net-(R9-Pad1) -> /UART1_RX
- U1 pad 16: /UART2_TX -> /ESP_UART1_RX
- U1 pad 17: /UART2_RX -> /ESP_UART1_TX
- U2 pad 3: Net-(D2-Pad2) -> Net-(D2-Pad1)
- U3 pad 1: +3.3V -> VBUS
Routing:
- net /EEP_SCL: track 125.6 -> 248.9 mm, vias 7 -> 9
- net VBUS: track 57.1 -> 179.0 mm, vias 2 -> 6
- net Net-(R22-Pad1): track 117.0 -> 0.00 mm, vias 6 -> 0
- net Net-(R21-Pad1): track 104.4 -> 0.00 mm, vias 4 -> 0
- net /EEP_SDA: track 130.6 -> 207.2 mm, vias 10 -> 13
- net /UART2_RX: track 72.0 -> 0.00 mm, vias 4 -> 0
- net /ESP_UART1_TX: track 151.4 -> 221.2 mm, vias 4 -> 10
- net /UART2_TX: track 45.2 -> 0.00 mm, vias 6 -> 0
- net /ESP_UART1_RX: track 114.9 -> 156.8 mm, vias 4 -> 8
- net Net-(R10-Pad1): track 40.3 -> 0.00 mm, vias 4 -> 0
- net Net-(R9-Pad1): track 40.0 -> 0.00 mm, vias 2 -> 0
- net GND: track 631.9 -> 607.9 mm, vias 106 -> 95
- net /UART1_RX: track 43.4 -> 52.7 mm
- net +3.3V: track 670.2 -> 661.2 mm, vias 51 -> 50
- net /UART1_TX: track 57.0 -> 64.4 mm
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- added copper zone on F.Cu, net GND
