File: hardware/EV6b/EV6 Board Design.kicad_pcb (KiCad board)
At the start: 4 copper layers, 72.7 x 89.4 mm, 116 parts, among them J1 Conn_01x02_Female, J10 Conn_01x08_Female, J11 Conn_01x06_Female, J12 Conn_01x04_Female, J13 Conn_01x04_Female, J14 Conn_01x04_Female, J15 Conn_01x02_Female, J2 Conn_01x02_Female, J3 Conn_01x04_Female, J4 Conn_01x08_Male, J5 Conn_01x04_Female, J6 Conn_01x04_Female, J7 Conn_01x04_Female, J8 Conn_01x06_Female, J9 USB_C_Receptacle, SW1 SW_Push, SW2 SW_Push, SW3 SW_Push, U1 STM32F405RGTx, U11 ESP32-S3-WROOM-1-N8R2, U12 MCP73832-2-OT, U13 BM14B(0.8)-24DS-0.4V(53), U2 AMS1117-3.3, U3 CH340C, U4 USBLC6-2P6, U5 STM32F091CCT6, U6 WM8960CGEFL/RV, Y1 Crystal_GND24

Commit message: Move to STM32F446
Parts:
- C2: value 22u -> 15u
- R40: value 1 -> 1R0
- R41: value 0 -> 1R0
- U1: value STM32F405RGTx -> STM32F446RET6
Changed lines of the file:
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@@
         (effects (font (size 1 1) (thickness 0.15)))
     )
-    (fp_text value "22u" (at 0 1.16 90) (layer "F.Fab") hide
+    (fp_text value "15u" (at 0 1.16 90) (layer "F.Fab") hide
         (effects (font (size 1 1) (thickness 0.15)))
     )
@@
         (effects (font (size 1 1) (thickness 0.15)))
     )
-    (fp_text value "STM32F405RGTx" (at 0 7.4) (layer "F.Fab") hide
+    (fp_text value "STM32F446RET6" (at 0 7.4) (layer "F.Fab") hide
         (effects (font (size 1 1) (thickness 0.15)))
     )
@@
         (effects (font (size 1 1) (thickness 0.15)))
     )
-    (fp_text value "0" (at 0 1.17) (layer "F.Fab") hide
+    (fp_text value "1R0" (at 0 1.17) (layer "F.Fab") hide
         (effects (font (size 1 1) (thickness 0.15)))
     )
@@
         (effects (font (size 1 1) (thickness 0.15)))
     )
-    (fp_text value "1" (at 0 1.17 90) (layer "F.Fab") hide
+    (fp_text value "1R0" (at 0 1.17 90) (layer "F.Fab") hide
         (effects (font (size 1 1) (thickness 0.15)))
     )
