File: hardware/EV9/EV9 Board Design.kicad_sch (KiCad schematic)
At the start: 111 parts, among them J1 Conn_01x02_Female, J10 Conn_01x08_Female, J11 Conn_01x06_Female, J12 Conn_01x04_Female, J13 Conn_01x04_Female, J14 Conn_01x04_Female, J15 Conn_01x02_Female, J2 Conn_01x02_Female, J3 Conn_01x04_Female, J4 Conn_01x08_Male, J5 Conn_01x04_Female, J6 Conn_01x04_Female, J7 Conn_01x04_Female, J8 Conn_01x06_Female, J9 USB_C_Receptacle, SW1 SW_Push, SW2 SW_Push, SW3 SW_Push, U1 STM32F405RGTx, U11 ESP32-S3-WROOM-1-N8R2, U12 MCP73832-2-OT, U13 BM14B(0.8)-24DS-0.4V(53), U2 AMS1117-3.3, U3 CH340C, U4 USBLC6-2P6, U5 STM32F030C8Tx, U6 WM8960CGEFL/RV, Y1 Crystal_GND24

Commit message: Removed LED, UI Serial, Net I2C connector/ changed button
Parts:
- removed J14, J3, J5: Conn_01x04_Female, 1x4 pin download:1x4pin 1mm connector, symbol Connector:Conn_01x04_Female
- removed R21: 1k5, Resistor_SMD:R_0402_1005Metric, symbol Device:R
- removed R33: 180, Resistor_SMD:R_0402_1005Metric, symbol Device:R
- removed R34, R35: 150, Resistor_SMD:R_0402_1005Metric, symbol Device:R
- removed SW1, SW2, SW3: SW_Push, Button_Switch_SMD:SW_DIP_SPSTx01_Slide_6.7x4.1mm_W6.73mm_P2.54mm_LowProfile_JPin, symbol Switch:SW_Push
- added C35: 100n, Capacitor_SMD:C_0402_1005Metric, symbol Device:C
- added R10: 4k7, Resistor_SMD:R_0402_1005Metric, symbol Device:R
- added SW4, SW5: SW_Push, Button_Switch_SMD:SW_DIP_SPSTx01_Slide_6.7x4.1mm_W6.73mm_P2.54mm_LowProfile_JPin, symbol Switch:SW_Push
- R20: value 1k5 -> 4k7; JLCPCB# C25867 -> C25900
Connections:
- net +3.3V: now also SW4.2
- net GND: now also C35.1, R10.1, SW5.2
- net MGMT_BOOT: now also R10.2, SW4.1
- net MGMT_NRST: now also R20.2, C35.2, SW5.1
- net NET_SCL: no longer names the net of U11.25 (IO48)
- net NET_SDA: no longer names the net of U11.24 (IO47)
- net NET_SDA: no longer R20.2
- net UI_RX3: no longer names the net of U1.30 (PB11)
- net UI_TX3: no longer names the net of U1.29 (PB10)
- no-connect marks 62 -> 66
Other:
- note added: "BOOT SW"
- note added: "NRST SW"
- note removed: "LED - 1MM T"
- note removed: "MGMT SW"
- note removed: "NET I2C - 1MM B"
- note removed: "UI SERIAL - 1MM B"
- title: EV8 - FINN BERG -> EV9 - FINN BERG
- moved on the sheet: J10, J13, R22, R26, R27, R28, R29, R30, R31
