File: hardware/EV10.1/EV10.1.kicad_sch (KiCad schematic)
At the start: 117 parts, among them J1 Conn_01x02_Socket, J10 Conn_01x08_Socket, J11 Conn_01x06_Female, J13 Conn_01x04_Female, J2 Conn_01x02_Female, J5 Conn_01x02_Socket, J7 Conn_01x04_Female, J8 Conn_01x06_Female, SW4 SW_Push, SW5 SW_Push, U1 STM32F405RGTx, U11 ESP32-S3-WROOM-1-N8R2, U13 BM14B(0.8)-24DS-0.4V(53), U2 BQ21040DBVR, U3 CH340C, U5 STM32F030C8Tx, U6 WM8960CGEFL/RV, U7 TPS63060, Y1 Crystal_GND24

Commit message: Added another test point to EV10.1 for BCLK. EV11 WIP
Parts:
- added TP13: P_I2S_BCLK, TestPoint:TestPoint_Keystone_5000-5004_Miniature, symbol Connector:TestPoint_Probe
- TP10: value P_UI_RX_NET -> P_UI_TX_NET
Connections:
- net I2S_BCLK: now also TP13.1
Changed lines of the file:
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@@
 	(wire
 		(pts
+			(xy 477.52 209.55) (xy 477.52 232.41)
+		)
+		(stroke
+			(width 0)
+			(type default)
+		)
+	)
+	(wire
+		(pts
 			(xy 67.31 111.76) (xy 67.31 113.03)
 		)
@@
 	(wire
 		(pts
+			(xy 430.53 209.55) (xy 477.52 209.55)
+		)
+		(stroke
+			(width 0)
+			(type default)
+		)
+	)
+	(wire
+		(pts
 			(xy 40.64 226.06) (xy 40.64 229.87)
 		)
@@
 		)
 	)
+	(label "I2S_BCLK"
+		(at 430.53 209.55 180)
+		(fields_autoplaced yes)
+		(effects
+			(font
+				(size 1.27 1.27)
+			)
+			(justify right bottom)
+		)
+	)
 	(label "LEDA_R"
 		(at 129.54 77.47 0)
@@
 			)
 		)
-		(property "Value" "P_UI_RX_NET"
+		(property "Value" "P_UI_TX_NET"
 			(at 445.4525 287.02 90)
 			(effects
@@
 					(unit 1)
 				)
+			)
+		)
+	)
+	(symbol
+		(lib_id "Connector:TestPoint_Probe")
+		(at 477.52 232.41 90)
+		(unit 1)
+		(exclude_from_sim no)
+		(in_bom yes)
+		(on_board yes)
+		(dnp no)
+		(property "Reference" "TP13"
+			(at 476.25 225.806 90)
+			(effects
+				(font
+					(size 1.27 1.27)
+				)
+			)
+		)
+		(property "Value" "P_I2S_BCLK"
+			(at 475.9325 227.33 90)
+			(effects
+				(font
+					(size 1.27 1.27)
+				)
+			)
+		)
+		(property "Footprint" "TestPoint:TestPoint_Keystone_5000-5004_Miniature"
+			(at 477.52 227.33 0)
+			(effects
+				(font
+					(size 1.27 1.27)
+				)
+				(hide yes)
+			)
+		)
+		(property "Datasheet" "~"
+			(at 477.52 227.33 0)
+			(effects
+				(font
+					(size 1.27 1.27)
+				)
+				(hide yes)
+			)
+		)
+		(property "Description" "test point (alternative probe-style design)"
+			(at 477.52 232.41 0)
+			(effects
+				(font
+					(size 1.27 1.27)
+				)
+				(hide yes)
+			)
+		)
+		(property "LCSC Part #" "C5199900"
+			(at 477.52 232.41 0)
+			(effects
+				(font
+					(size 1.27 1.27)
+				)
+				(hide yes)
+			)
+		)
+		(pin "1"
+		)
+		(instances
+			(project "EV10.1"
+				(path "/bd865368-262b-4f76-b7a6-1673c2cb0f8c"
+					(reference "TP13")
+					(unit 1)
+				)
