File: hardware/EV10.1/EV10.1.kicad_pcb (KiCad board)
At the start: 4 copper layers, 72.7 x 89.4 mm, 123 parts, among them J1 Conn_01x02_Socket, J10 Conn_01x08_Socket, J11 Conn_01x06_Female, J13 Conn_01x04_Female, J2 Conn_01x02_Female, J5 Conn_01x02_Socket, J7 Conn_01x04_Female, J8 Conn_01x06_Female, SW4 SW_Push, SW5 SW_Push, U1 STM32F405RGTx, U11 ESP32-S3-WROOM-1-N8R2, U13 BM14B(0.8)-24DS-0.4V(53), U2 BQ21040DBVR, U3 CH340C, U5 STM32F030C8Tx, U6 WM8960CGEFL/RV, U7 TPS63060, Y1 Crystal_GND24

Commit message: changes before submit 10.1
Parts:
- removed REF** (x5): MountingHole_2.1mm, MountingHole:MountingHole_2.1mm
- C29, C30: value 100U -> 100u
- C37, C40, C42: value 0.1u -> 100n
- J11, J8: value Conn_01x06_Female -> Conn_01x06_Socket
- J13, J7: value Conn_01x04_Female -> Conn_01x04_Socket
- J2: value Conn_01x02_Female -> Conn_01x02_Socket
- TP1: value P_USB_TX_MGMT -> TP
- TP10: value P_UI_TX_NET -> TP
- TP11: value P_UI_RX_NET -> TP
- TP12: value P_GND -> TP
- TP13: value P_I2S_BCLK -> TP
- TP2: value P_USB_RX_MGMT -> TP
- TP3: value P_I2S_ADCDAT -> TP
- TP4: value P_I2S_DACDAT -> TP
- TP5: value P_I2S_DACLRC -> TP
- TP6: value P_UI_TX_MGMT -> TP
- TP7: value P_UI_RX_MGMT -> TP
- TP8: value P_NET_TX_MGMT -> TP
- TP9: value P_NET_RX_MGMT -> TP
- U2: footprint BQ21040DBVR:SOT95P280X145-6N -> Package_TO_SOT_SMD:SOT-23-6
- moved R26 0.55 mm to (129.3, 139.9)
- moved C1 0.38 mm to (134.3, 139.9)
- moved R22 0.29 mm to (134.2, 135.5)
Connections:
- U1 pad 14: /BATTERY_MON -> unconnected-(U1-PA0-Pad14)
Routing:
- net /BATTERY_MON: track 28.6 -> 0.00 mm
- net GND: track 572.3 -> 575.9 mm, vias 154 -> 155
- net /KB_MIC: track 49.4 -> 50.9 mm
- net Net-(U6-HP_L): track 7.26 -> 5.76 mm
- net /NET_RST: track 57.2 -> 56.3 mm
- net /KB_COL5: track 28.2 -> 27.4 mm
- net Net-(U2-ISET): track 1.25 -> 1.80 mm
Other:
- board text added: "2024-04"
- board text removed: "2024-03"
