File: hardware/EV12/EV12 Board Design.kicad_sch (KiCad schematic)
At the start: 129 parts, among them CN2 Conn_05x02_Female, CN3 Conn_01x06_Female, CN4 Conn_01x06_Female, CN5 Conn_02x05_Male, CN6 Conn_02x05_Male, CN7 Conn_02x05_Male, J1 Conn_01x02_Socket, J10 Conn_01x08_Socket, J2 AudioJack1, J3 Conn_01x06_Socket, J9 USB_C_Receptacle, SW1 SW_Push, SW2 SW_Push, SW4 SW_Push, SW5 SW_Push, SW6 SW_SPDT, U1 STM32F405RGTx, U11 ESP32-S3-WROOM-1-N8R2, U13 BM14B(0.8)-24DS-0.4V(53), U2 BQ21040DBV, U3 CH340C, U4 USBLC6-2P6, U5 M24C02-RMN6TP, U6 WM8960CGEFL/RV, U7 TPS63060, U8 STM32F072CBTx, Y1 Crystal_GND24

Commit message: Updated Field Information
Parts:
- CN2, CN5, CN6, CN7: JLCPCB# C2962219 -> (none)
- D3, D4, D5, D7: JLCPCB# C2874115 -> (none)
- J2: MPN PJ-320D -> (none)

Commit message: chore: Update ft fields to match their new expected field names
Parts:
- CN3, CN4, J1, J3: FT Rotation Offset (none) -> 180; JLCPCB Rotation Offset 180 -> (none)
- J10: FT Position Offset (none) -> 0,-0.1270; JLCPCB Position Offset 0,-0.1270 -> (none)
- J2: FT Position Offset (none) -> 0.889,0; FT Rotation Offset (none) -> 90; JLCPCB Position Offset 0.889,0 -> (none); JLCPCB Rotation Offset 90 -> (none)
- J9: FT Position Offset (none) -> 0,1.397; JLCPCB Position Offset 0,1.397 -> (none)
- SW6: FT Position Offset (none) -> 0,0; JLCPCB Position Offset 0,-3.556 -> (none)
- U11: FT Position Offset (none) -> 0,-0.508; JLCPCB Position Offset 0,-0.508 -> (none)
- U13: FT Position Offset (none) -> 2.9800,1.2065; JLCPCB Position Offset 2.9800,1.2065 -> (none)
- U4, U7: FT Rotation Offset (none) -> 270; JLCPCB Rotation Offset 270 -> (none)
- U6: FT Rotation Offset (none) -> -90; JLCPCB Rotation Offset -90 -> (none)
