File: hardware/EV14/ev14_board_design/ev14_board_design.kicad_sch (KiCad schematic)
At the start: 154 parts, among them CN1 Conn_05x02_Female, J1 USB_C_Receptacle, J2 Conn_01x02_Socket, J3 Conn_02x03_Odd_Even, J4 Conn_01x08_Socket, J5 AudioJack4, J6 AudioJack4, Q1 2N7002, SW1 SW_SPDT, SW2 SW_Push, SW3 SW_Push, SW4 SW_Push, SW5 SW_Push, U1 BQ21040DBV, U10 STM32F405RGTx, U2 USBLC6-2P6, U3 STM32F072CBTx, U4 CH340C, U5 TPS63060, U6 ESP32-S3-WROOM-1, U7 WM8960CGEFL/RV, U8 M24C02-RMN6TP, U9 BM14B(0.8)-24DS-0.4V(53), Y1 Crystal_GND24

Commit message: Updated ev14 with audio added
Parts:
- removed J4: Conn_01x08_Socket, Hactar_Footprints:CONN-SMD_8P-P2.00_S8B-PH-SM4-TB-LF-SN, symbol Connector:Conn_01x08_Socket
- added J7: Conn_01x35_Socket, Hactar_Footprints:CONN-SMD_HCTL_HC-FPC-03-09-35RLTAG, symbol Connector:Conn_01x35_Socket
Connections:
- net +3.3V: now also J7.28 (Pin_28), J7.29 (Pin_29)
- net DISP_BL: now also J7.31 (Pin_31)
- net DISP_CLK: now also J7.3 (Pin_3)
- net DISP_CS: now also J7.2 (Pin_2)
- net DISP_DC: now also J7.1 (Pin_1)
- net DISP_MOSI: now also J7.5 (Pin_5)
- net DISP_RST: now also J7.6 (Pin_6)
- net GND: now also J7.27 (Pin_27), J7.30 (Pin_30), J7.32 (Pin_32), J7.33 (Pin_33), J7.34 (Pin_34)
- net LEDB_G: now also R24.1; no longer R24.2
- net at D5.4 (-): now also R24.2; no longer R24.1
- net D_P: now reaches J1.A6 (D+), J1.B6 (D+), U2.4 (I/O2)
- net D_N: now reaches J1.A7 (D-), J1.B7 (D-), U2.6 (I/O1)
- net UD_N: now reaches U2.1 (I/O1), U4.6 (UD-)
- net UD_P: now reaches U2.3 (I/O2), U4.5 (UD+)
- net UI_RX2_NET renamed UI_RX2_NET_-
- net UI_TX2_NET renamed UI_TX2_NET_+
- no-connect marks 32 -> 54
Other:
- note added: "Display - 0.3mm FPC"
- note removed: "Display - 2MM B"
- moved on the sheet: R24

Commit message: Fet array for analog jack switching
Parts:
- added C48: 100u, Capacitor_SMD:C_1206_3216Metric, symbol Device:C_Small
- added J10, J7, J8, J9: Conn_02x05_Counter_Clockwise, Hactar_Footprints:HDR-SMD_10P-P2.54-V-F-R2-C5-LS7.1-1, symbol Connector_Generic:Conn_02x05_Counter_Clockwise
- added Q2: Q_Dual_NMOS_S1G1D2S2G2D1, Hactar_Footprints:SOT-363_L2.1-W1.3-P0.65-LS2.3-BL, symbol Transistor_FET:Q_Dual_NMOS_S1G1D2S2G2D1
- added Q3: PMOS, Hactar_Footprints:SOT-23-3_L2.9-W1.3-P1.90-LS2.4-BR, symbol Simulation_SPICE:PMOS
- added R63, R70, R71, R72, R73, R74: 1k0, Resistor_SMD:R_0402_1005Metric, symbol Device:R_US
- added R64: 47k, Resistor_SMD:R_0402_1005Metric, symbol Device:R_Small_US
- added R65: 100k, Resistor_SMD:R_0402_1005Metric, symbol Device:R_US
- added R66, R67, R68, R69: 4k7, Resistor_SMD:R_0402_1005Metric, symbol Device:R_US
- renumbered C33 to C32, C34 to C33, C35 to C34, C32 to C35, C38 to C37, C37 to C38, J5 to J3, J6 to J4, J3 to J5, J7 to J6, R32 to R31, R33 to R32, R31 to R33, R47 to R36, R48 to R37, R36 to R38, R37 to R39, R38 to R40, R39 to R41, R40 to R42, R41 to R43, R42 to R44, R43 to R45, R44 to R46, R45 to R47, R46 to R48, TP3 to TP1, TP4 to TP2, TP5 to TP3, TP6 to TP4, U7 to U6, U6 to U7
Connections:
- net +3.3V: now also J7.1 (Pin_1), J8.1 (Pin_1)
- net GND: now also J10.5 (Pin_5), J10.6 (Pin_6), J7.2 (Pin_2), J8.2 (Pin_2), R64.2, R66.2, R67.2, R68.2, R69.2
- net GNDA: now also Q2.1 (S), R65.1; no longer J3.S
- net I2S_ADCDAT: now also J8.6 (Pin_6), R66.1
- net I2S_BCLK: now also J8.4 (Pin_4), R69.1
- net I2S_DACDAT: now also J8.7 (Pin_7), R68.1
- net I2S_DACLRC: now also J8.5 (Pin_5), R67.1
- net MCLK: now also J8.10 (Pin_10), R64.1
- net MGMT_BOOT: now also J10.7 (Pin_7)
- net MGMT_DEBUG_1: now also J9.10 (Pin_10)
- net MGMT_DEBUG_2: now also J9.9 (Pin_9)
- net MGMT_NRST: now also J10.8 (Pin_8)
- net MGMT_SWCLK: now also J10.10 (Pin_10)
- net MGMT_SWDIO: now also J10.9 (Pin_9)
- net MIC_N: now also J3.R2
- net MIC_P: now also Q2.4 (S), Q3.3 (S); no longer J4.T
- net NET_BOOT: now also J10.1 (Pin_1)
- net NET_DEBUG_1: now also R70.1
- net NET_DEBUG_2: now also R71.1
- net NET_DEBUG_3: now also R72.1
- net NET_NRST: now also J10.4 (Pin_4)
- net NET_RX1_MGMT: now also J10.3 (Pin_3), J7.7 (Pin_7)
- net NET_TX1_MGMT: now also J10.2 (Pin_2), J7.6 (Pin_6)
- net UI_CTS1_MGMT: now also J9.4 (Pin_4)
- net UI_DEBUG_1: now also R74.2
- net UI_DEBUG_2: now also R73.2
- net UI_RTS1_MGMT: now also J9.5 (Pin_5)
- net UI_RX1_MGMT: now also J7.9 (Pin_9)
- net UI_RX2_NET_-: no longer U10.17 (PA3)
- net UI_SCL: now also J8.8 (Pin_8)
- net UI_SDA: now also J8.9 (Pin_9)
- net UI_TX1_MGMT: now also J7.8 (Pin_8)
- net UI_TX2_NET_+: no longer U10.16 (PA2)
- net USB_RX1_MGMT: now also J7.10 (Pin_10)
- net USB_TX1_MGMT: now also J7.5 (Pin_5)
- net at U6.29 (HP_R): now also C48.1
- net HP_R: now reaches J3.R1
- net HP_R: now also C48.2, R65.2
- new net: Q2.2 (G), Q2.5 (G), Q3.2 (G), R63.1
- new net: J4.T, Q2.3 (D), R63.2
- new net: J3.S, Q2.6 (D), Q3.1 (D)
- new net: J9.6 (Pin_6), R70.2
- new net: J9.8 (Pin_8), R72.2
- new net: J9.2 (Pin_2), R74.1
- new net: J9.3 (Pin_3), R73.1
- new net: J9.7 (Pin_7), R71.2
- new net UI_RX2_NET: J7.4 (Pin_4), U10.17 (PA3)
- new net UI_TX2_NET: J7.3 (Pin_3), U10.16 (PA2)
- no-connect marks 54 -> 53
Other:
- note added: "D1"
- note added: "D2"
- note added: "DEBUG"
- note added: "Default mode (3.5mm only): 3.5mm jack: S = MIP_P, R2 = MIC_N, R1 = HP_R, T = HP_L 2.5mm jack: S = MIC_N, T = 0V"
- note added: "Detect"
- note added: "Dual jack mode (3.5mm and 2.5mm): 3.5mm jack: S = GNDA, R2 = MIC_N, R1 = HP_R, T = HP_L 2.5mm jack: S = MIC_N, T =! 0V = MIC_P"
- note added: "G1"
- note added: "G2"
- note added: "GPIO DEBUG"
- note added: "I2S + I2C DEBUG"
- note added: "MOSFET ARRAY"
- note added: "NET SERIAL UPLOADER + MGMT ST LINK"
- note added: "S1"
- note added: "S2"
- note added: "SERIAL DEBUG"
- note removed: "Dual Headset T"
- moved on the sheet: C21, C23, C25, C26, C28, C32, C33, C34, C36, C37, C38, C39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

Commit message: Latest version of Ev14
Changed lines of the file:
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@@
 	)
 	(junction
-		(at 299.72 191.77)
-		(diameter 0)
-		(color 0 0 0 0)
-	)
-	(junction
 		(at 265.43 351.79)
 		(diameter 0)
@@
 	)
 	(junction
-		(at 298.45 191.77)
-		(diameter 0)
-		(color 0 0 0 0)
-	)
-	(junction
 		(at 40.64 68.58)
 		(diameter 0)
@@
 	)
 	(junction
-		(at 304.8 191.77)
-		(diameter 0)
-		(color 0 0 0 0)
-	)
-	(junction
 		(at 57.15 240.03)
 		(diameter 0)
@@
 	)
 	(junction
-		(at 298.45 190.5)
-		(diameter 0)
-		(color 0 0 0 0)
-	)
-	(junction
 		(at 240.03 170.18)
 		(diameter 0)
@@
 	(wire
 		(pts
-			(xy 304.8 191.77) (xy 299.72 191.77)
-		)
-		(stroke
-			(width 0)
-			(type default)
-		)
-	)
-	(wire
-		(pts
 			(xy 464.82 214.63) (xy 464.82 213.36)
 		)
@@
 	(wire
 		(pts
-			(xy 298.45 191.77) (xy 297.18 191.77)
-		)
-		(stroke
-			(width 0)
-			(type default)
-		)
-	)
-	(wire
-		(pts
 			(xy 250.19 181.61) (xy 245.11 181.61)
 		)
@@
 	(wire
 		(pts
-			(xy 299.72 191.77) (xy 299.72 190.5)
-		)
-		(stroke
-			(width 0)
-			(type default)
-		)
-	)
-	(wire
-		(pts
 			(xy 265.43 226.06) (xy 279.4 226.06)
 		)
@@
 	(wire
 		(pts
-			(xy 299.72 191.77) (xy 298.45 191.77)
-		)
-		(stroke
-			(width 0)
-			(type default)
-		)
-	)
-	(wire
-		(pts
 			(xy 214.63 229.87) (xy 228.6 229.87)
 		)
@@
 	(wire
 		(pts
-			(xy 298.45 191.77) (xy 298.45 190.5)
-		)
-		(stroke
-			(width 0)
-			(type default)
-		)
-	)
-	(wire
-		(pts
 			(xy 553.72 91.44) (xy 558.8 91.44)
 		)
@@
 	(wire
 		(pts
-			(xy 299.72 190.5) (xy 298.45 190.5)
-		)
-		(stroke
-			(width 0)
-			(type default)
-		)
-	)
-	(wire
-		(pts
 			(xy 219.71 322.58) (xy 227.33 322.58)
 		)
@@
 		)
 	)
-	(wire
-		(pts
-			(xy 297.18 190.5) (xy 298.45 190.5)
-		)
-		(stroke
-			(width 0)
-			(type default)
-		)
-	)
 	(polyline
 		(pts
@@
 	(wire
 		(pts
-			(xy 297.18 191.77) (xy 297.18 190.5)
-		)
-		(stroke
-			(width 0)
-			(type default)
-		)
-	)
-	(wire
-		(pts
 			(xy 213.36 336.55) (xy 213.36 340.36)
 		)
@@
 		(on_board yes)
 		(dnp no)
-		(fields_autoplaced yes)
 		(property "Reference" "H1"
 			(at 149.86 226.0599 0)
@@
 		)
 		(property "Value" "MountingHole"
-			(at 149.86 228.5999 0)
+			(at 149.86 228.6 0)
 			(effects
 				(font
