File: hardware/EV14/ev14_board_design/ev14_board_design.kicad_pcb (KiCad board)
At the start: 4 copper layers, 50 x 80 mm, 154 parts, among them CN1 Conn_05x02_Female, J1 USB_C_Receptacle, J2 Conn_01x02_Socket, J3 Conn_02x03_Odd_Even, J4 Conn_01x08_Socket, J5 AudioJack4, J6 AudioJack4, Q1 2N7002, SW1 SW_SPDT, SW2 SW_Push, SW3 SW_Push, SW4 SW_Push, SW5 SW_Push, U1 BQ21040DBV, U10 STM32F405RGTx, U2 USBLC6-2P6, U3 STM32F072CBTx, U4 CH340C, U5 TPS63060, U6 ESP32-S3-WROOM-1, U7 WM8960CGEFL/RV, U8 M24C02-RMN6TP, U9 BM14B(0.8)-24DS-0.4V(53), Y1 Crystal_GND24

Commit message: Updated ev14 with audio added
Parts:
- removed J4: Conn_01x08_Socket, Hactar_Footprints:CONN-SMD_8P-P2.00_S8B-PH-SM4-TB-LF-SN
- added J7: Conn_01x35_Socket, Hactar_Footprints:CONN-SMD_HCTL_HC-FPC-03-09-35RLTAG, F.Cu at (199.9, 93.8)
- moved C35 289.3 mm to (214.4, 55.8), turned to 90 degrees
- moved NT1 286.2 mm to (213.3, 65.8), turned to 90 degrees
- moved Q1 269.5 mm to (220.3, 114.5), turned to -90 degrees
- moved D7 263.2 mm to (187.3, 64.5), turned to 180 degrees
- moved CN1 254.7 mm to (213.0, 92.0)
- moved L1 248.8 mm to (208.8, 65.5)
- moved JP2 243.4 mm to (208.1, 54.5), turned to 180 degrees
- moved J3 211.6 mm to (218.9, 122.6), turned to 90 degrees
- moved J5 136.7 mm to (199.3, 60.5)
- moved R33 117.8 mm to (212.7, 55.8), turned to 90 degrees
- moved J6 116.5 mm to (189.3, 58.3)
- moved R15 115.6 mm to (222.3, 107.8), turned to 180 degrees
- moved R32 115.0 mm to (210.6, 55.8), turned to -90 degrees
- moved R23 113.1 mm to (222.8, 106.8), turned to 180 degrees
- moved R25 112.0 mm to (221.8, 112.0)
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Connections:
- net /UI_RX2_NET renamed /UI_RX2_NET_-
- net /UI_TX2_NET renamed /UI_TX2_NET_+
- net Net-(J1-D+-PadA6) renamed /D_P
- net Net-(J1-D--PadA7) renamed /D_N
- net Net-(U4-UD+) renamed /UD_P
- net Net-(U4-UD-) renamed /UD_N
- R24 pad 1: Net-(D5---Pad4) -> /LEDB_G
- R24 pad 2: /LEDB_G -> Net-(D5---Pad4)
Routing:
- net +3.3VA: track 0.00 -> 75.1 mm, vias 0 -> 5
- net GND: track 82.0 -> 151.6 mm, vias 74 -> 87
- net /MCLK: track 0.00 -> 59.2 mm
- net +3.3V: track 15.5 -> 59.6 mm, vias 14 -> 25
- net /UI_SDA: track 0.00 -> 43.6 mm, vias 0 -> 2
- net /I2S_DACDAT: track 0.00 -> 43.1 mm, vias 0 -> 2
- net /UI_SCL: track 0.00 -> 42.7 mm, vias 0 -> 2
- net /I2S_ADCDAT: track 0.00 -> 41.8 mm, vias 0 -> 2
- net /I2S_BCLK: track 0.00 -> 40.2 mm
- net /I2S_DACLRC: track 0.00 -> 39.2 mm
- net /MIC_P: track 0.00 -> 37.7 mm
- net Net-(D4---Pad3): track 0.00 -> 37.6 mm
- net Net-(D5---Pad1): track 0.00 -> 36.2 mm, vias 0 -> 2
- net Net-(D4---Pad4): track 0.00 -> 33.1 mm
- net /UI_NRST: track 0.00 -> 32.8 mm, vias 0 -> 2
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- added copper zone on B.Cu, net GNDA
- added copper zone on F.Cu, net GNDA
- added copper zone on In1.Cu, net GNDA
- added copper zone on In2.Cu, net GNDA

Commit message: Fet array for analog jack switching
Parts:
- added C48: 100u, Capacitor_SMD:C_1206_3216Metric, F.Cu at (216.7, 57.3)
- added J10: Conn_02x05_Counter_Clockwise, Hactar_Footprints:HDR-SMD_10P-P2.54-V-F-R2-C5-LS7.1-1, F.Cu at (231.1, 123.5)
- added J7: Conn_02x05_Counter_Clockwise, Hactar_Footprints:HDR-SMD_10P-P2.54-V-F-R2-C5-LS7.1-1, F.Cu at (242.4, 108.6)
- added J8: Conn_02x05_Counter_Clockwise, Hactar_Footprints:HDR-SMD_10P-P2.54-V-F-R2-C5-LS7.1-1, F.Cu at (231.0, 108.6)
- added J9: Conn_02x05_Counter_Clockwise, Hactar_Footprints:HDR-SMD_10P-P2.54-V-F-R2-C5-LS7.1-1, F.Cu at (242.2, 123.4)
- added Q2: Q_Dual_NMOS_S1G1D2S2G2D1, Hactar_Footprints:SOT-363_L2.1-W1.3-P0.65-LS2.3-BL, F.Cu at (182.9, 58.0)
- added Q3: PMOS, Hactar_Footprints:SOT-23-3_L2.9-W1.3-P1.90-LS2.4-BR, F.Cu at (182.9, 55.2)
- added R63: 1k0, Resistor_SMD:R_0402_1005Metric, F.Cu at (185.5, 56.4)
- added R64: 47k, Resistor_SMD:R_0402_1005Metric, F.Cu at (327.3, 95.7)
- added R65: 100k, Resistor_SMD:R_0402_1005Metric, F.Cu at (215.5, 54.4)
- added R66: 4k7, Resistor_SMD:R_0402_1005Metric, F.Cu at (327.3, 97.7)
- added R67: 4k7, Resistor_SMD:R_0402_1005Metric, F.Cu at (327.3, 99.7)
- added R68: 4k7, Resistor_SMD:R_0402_1005Metric, F.Cu at (327.3, 101.7)
- added R69: 4k7, Resistor_SMD:R_0402_1005Metric, F.Cu at (327.3, 103.7)
- added R70: 1k0, Resistor_SMD:R_0402_1005Metric, F.Cu at (330.2, 95.7)
- added R71: 1k0, Resistor_SMD:R_0402_1005Metric, F.Cu at (330.2, 97.7)
- added R72: 1k0, Resistor_SMD:R_0402_1005Metric, F.Cu at (330.2, 99.7)
- added R73: 1k0, Resistor_SMD:R_0402_1005Metric, F.Cu at (330.2, 101.7)
- added R74: 1k0, Resistor_SMD:R_0402_1005Metric, F.Cu at (330.2, 103.7)
- moved U9 235.2 mm to (199.6, 115.8), turned to 90 degrees
- moved SW3 189.7 mm to (176.5, 100.8), turned to -90 degrees
- moved SW2 183.4 mm to (176.5, 109.6), turned to -90 degrees
- moved TP3 127.8 mm to (104.5, 60.0)
- moved TP4 127.8 mm to (104.5, 64.1)
- moved TP1 127.8 mm to (100.5, 60.0)
- moved TP2 127.8 mm to (100.5, 64.1)
- moved R3 118.9 mm to (222.8, 105.7), turned to 180 degrees
- moved R4 109.2 mm to (211.6, 96.9), turned to 90 degrees
- moved R5 108.5 mm to (210.6, 96.9), turned to 90 degrees
- moved R39 108.0 mm to (219.9, 111.2), turned to -90 degrees
- moved R38 106.7 mm to (218.8, 111.2), turned to -90 degrees
- moved R2 105.8 mm to (210.0, 111.3), turned to -90 degrees
- moved C17 103.9 mm to (212.8, 125.2), turned to 180 degrees
- moved R22 103.2 mm to (212.8, 124.2)
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- renumbered C33 to C32, C34 to C33, C35 to C34, C32 to C35, C38 to C37, C37 to C38, J5 to J3, J6 to J4, J3 to J5, J7 to J6, R32 to R31, R33 to R32, R31 to R33, R47 to R36, R48 to R37, R36 to R38, R37 to R39, R38 to R40, R39 to R41, R40 to R42, R41 to R43, R42 to R44, R43 to R45, R44 to R46, R45 to R47, R46 to R48, TP3 to TP1, TP4 to TP2, TP5 to TP3, TP6 to TP4, U7 to U6, U6 to U7
Connections:
- J3 pad R1: unconnected-(J5-PadR1) -> /HP_R
- J3 pad R2: unconnected-(J5-PadR2) -> /MIC_N
- J3 pad S: GNDA -> Net-(Q2A-D)
- J4 pad T: /MIC_P -> Net-(Q2B-D)
- U10 pad 16: /UI_TX2_NET_+ -> /UI_TX2_NET
- U10 pad 17: /UI_RX2_NET_- -> /UI_RX2_NET
- U6 pad 29: unconnected-(U7-HP_R-Pad29) -> Net-(U6-HP_R)
Routing:
- net /MGMT_BOOT: track 0.00 -> 88.7 mm, vias 0 -> 3
- net /UI_RTS1_MGMT: track 2.64 -> 86.8 mm, vias 0 -> 2
- net /MGMT_NRST: track 0.00 -> 83.3 mm, vias 0 -> 3
- net /UI_CTS1_MGMT: track 2.77 -> 82.6 mm, vias 0 -> 2
- net Net-(D3-A): track 13.7 -> 86.9 mm, vias 0 -> 2
- net /UI_TX1_MGMT: track 4.58 -> 74.3 mm, vias 0 -> 2
- net /UI_RX1_MGMT: track 4.15 -> 73.6 mm, vias 0 -> 2
- net /UI_SDA: track 43.6 -> 108.1 mm, vias 2 -> 4
- net /UI_NRST: track 32.8 -> 95.8 mm, vias 2 -> 6
- net /UI_SCL: track 42.7 -> 104.7 mm, vias 2 -> 4
- net /UI_RTS2_NET: track 0.00 -> 55.3 mm, vias 0 -> 4
- net /UI_SWDIO: track 8.53 -> 62.7 mm, vias 1 -> 2
- net /UI_CTS2_NET: track 0.00 -> 54.2 mm, vias 0 -> 4
- net /NET_READY: track 0.00 -> 50.8 mm, vias 0 -> 6
- net /NET_NRST: track 1.60 -> 48.1 mm, vias 0 -> 2
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Other:
- board size 50 x 80 mm -> 75 x 80 mm

Commit message: Latest version of Ev14
Parts:
- moved R70 118.4 mm to (216.3, 63.5), turned to -90 degrees
- moved R71 118.0 mm to (217.3, 63.5), turned to -90 degrees
- moved R72 117.6 mm to (218.3, 63.5), turned to -90 degrees
- moved R64 114.8 mm to (212.5, 96.8), turned to 90 degrees
- moved R66 113.8 mm to (213.5, 96.8), turned to 90 degrees
- moved R74 112.9 mm to (217.5, 96.8), turned to 90 degrees
- moved R68 112.9 mm to (214.5, 96.8), turned to 90 degrees
- moved R69 112.0 mm to (215.5, 96.8), turned to 90 degrees
- moved R73 111.8 mm to (218.5, 96.8), turned to 90 degrees
- moved R67 110.8 mm to (216.5, 96.8), turned to 90 degrees
- moved TP3 79.0 mm to (167.7, 107.5)
- moved TP2 78.2 mm to (167.6, 104.2)
- moved TP1 77.8 mm to (164.4, 104.3)
- moved TP4 74.4 mm to (164.7, 107.8)
- moved R12 26.5 mm to (184.3, 101.0), turned to 180 degrees
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Routing:
- net /UI_RX2_NET: track 0.00 -> 101.0 mm, vias 0 -> 2
- net /UI_TX2_NET: track 0.00 -> 101.0 mm, vias 0 -> 2
- net /NET_TX1_MGMT: track 0.00 -> 73.1 mm, vias 0 -> 6
- net /UI_BOOT0: track 1.67 -> 74.2 mm, vias 0 -> 4
- net /MCLK: track 57.9 -> 130.1 mm, vias 0 -> 2
- net /NET_RX1_MGMT: track 0.00 -> 71.3 mm, vias 0 -> 4
- net Net-(J9-Pin_8): track 0.00 -> 69.7 mm, vias 0 -> 2
- net GNDA: track 31.4 -> 98.1 mm, vias 6 -> 7
- net Net-(J9-Pin_7): track 0.00 -> 66.4 mm, vias 0 -> 2
- net Net-(J9-Pin_6): track 0.00 -> 61.6 mm, vias 0 -> 2
- net /PTT_AI_BTN: track 4.44 -> 63.1 mm, vias 1 -> 4
- net /I2S_BCLK: track 39.5 -> 97.9 mm, vias 0 -> 2
- net /I2S_DACDAT: track 42.4 -> 100.3 mm, vias 2 -> 4
- net /UI_DEBUG_1: track 0.00 -> 57.3 mm, vias 0 -> 2
- net /I2S_DACLRC: track 38.8 -> 94.4 mm, vias 0 -> 2
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Other:
- board size 75 x 80 mm -> 75.2 x 80 mm

Commit message: Latest version of EV14
Routing:
- net GND: track 194.1 -> 232.4 mm, vias 92 -> 95
- net +3.3V: track 96.1 -> 134.3 mm, vias 30 -> 33
- net /UI_SDA: track 137.8 -> 141.3 mm
- net /UI_SCL: track 137.9 -> 138.6 mm
