File: hardware/jack_breakout/jack_breakout.kicad_sch (KiCad schematic)
At the start: 4 parts, among them CN1 PJ-242, J1 3.5mm, J2 Conn_01x06_Socket, J3 Conn_01x04_Socket

Commit message: chore: add jlcpcb part numbers
Parts:
- J2: footprint Connector_PinHeader_2.54mm:PinHeader_1x06_P2.54mm_Vertical -> Connector_PinSocket_2.54mm:PinSocket_1x06_P2.54mm_Vertical
- J3: footprint Connector_PinHeader_2.54mm:PinHeader_1x04_P2.54mm_Vertical -> Connector_PinSocket_2.54mm:PinSocket_1x04_P2.54mm_Vertical
Changed lines of the file:
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@@
 			)
 		)
-		(property "Footprint" "Connector_PinHeader_2.54mm:PinHeader_1x06_P2.54mm_Vertical"
+		(property "Footprint" "Connector_PinSocket_2.54mm:PinSocket_1x06_P2.54mm_Vertical"
 			(at 50.8 27.94 0)
 			(effects
@@
 			)
 		)
-		(property "Footprint" "Connector_PinHeader_2.54mm:PinHeader_1x04_P2.54mm_Vertical"
+		(property "Footprint" "Connector_PinSocket_2.54mm:PinSocket_1x04_P2.54mm_Vertical"
 			(at 50.8 46.99 0)
 			(effects

Commit message: chore: add missing jlcpcb numbers and rotations
Parts:
- J2: JLCPCB Part # (none) -> C2832269
- J3: JLCPCB Part # (none) -> C18078127
Changed lines of the file:
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@@
+			)
+		)
+		(property "JLCPCB Part #" "C2832269"
+			(at 50.8 27.94 0)
+			(effects
+				(font
+					(size 1.27 1.27)
+				)
+				(hide yes)
 			)
 		)
@@
 			(at 50.8 46.99 0)
 			(effects
+				(font
+					(size 1.27 1.27)
+				)
+				(hide yes)
+			)
+		)
+		(property "JLCPCB Part #" "C18078127"
+			(at 50.8 46.99 0)
+			(effects

Commit message: Jack breakout (#305)
* feat: make jack breakout

* chore: add jlcpcb part numbers

* chore small cleanup
Parts:
- J2: JLCPCB Part # C2832269 -> (none)
- J3: JLCPCB Part # C18078127 -> (none)
Changed lines of the file:
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@@
-			)
-		)
-		(property "JLCPCB Part #" "C2832269"
-			(at 50.8 27.94 0)
-			(effects
-				(font
-					(size 1.27 1.27)
-				)
-				(hide yes)
 			)
 		)
@@
 			(at 50.8 46.99 0)
 			(effects
-				(font
-					(size 1.27 1.27)
-				)
-				(hide yes)
-			)
-		)
-		(property "JLCPCB Part #" "C18078127"
-			(at 50.8 46.99 0)
-			(effects
