File: hardware/ev14/ev14.kicad_sch (KiCad schematic)
At the start: 173 parts, among them CN1 Conn_05x02_Female, J1 USB_C_Receptacle, J10 Conn_02x05_Counter_Clockwise, J2 Conn_01x02_Socket, J3 AudioJack4, J4 AudioJack4, J5 Conn_02x03_Odd_Even, J6 Conn_01x35_Socket, J7 Conn_02x05_Counter_Clockwise, J8 Conn_02x05_Counter_Clockwise, J9 Conn_02x05_Counter_Clockwise, Q1 2N7002, Q2 Q_Dual_NMOS_S1G1D2S2G2D1, Q3 PMOS, SW1 SW_SPDT, SW2 SW_Push, SW3 SW_Push, SW4 SW_Push, SW5 SW_Push, U1 BQ21040DBV, U10 STM32F405RGTx, U2 USBLC6-2P6, U3 STM32F072CBTx, U4 CH340C, U5 TPS63060, U6 WM8960CGEFL/RV, U7 ESP32-S3-WROOM-1, U8 M24C02-RMN6TP, U9 BM14B(0.8)-24DS-0.4V(53), Y1 Crystal_GND24

Commit message: First finished draft of Ev14
Parts:
- removed TP1, TP2, TP3, TP4: TestPoint, TestPoint:TestPoint_THTPad_D2.0mm_Drill1.0mm, symbol Connector:TestPoint
Connections:
- net UI_RX2_NET_- is gone; now on net UI_RX2_NET: U7.10 (IO17)
- net UI_TX2_NET_+ is gone; now on net UI_TX2_NET: U7.11 (IO18)
- net KB_LEDA_1&2: no longer names the net of U9.26
- net KB_LEDA_3&4: no longer names the net of U9.24
- net KB_LEDK_1&4: no longer names the net of U9.25
- net KB_LEDK_2&3: no longer names the net of U9.23
- no-connect marks 53 -> 57

Commit message: Updated complete EV14 draft
Parts:
- added J11: Conn_02x05_Counter_Clockwise, Hactar_Footprints:HDR-SMD_10P-P2.54-V-F-R2-C5-LS7.1-1, symbol Connector_Generic:Conn_02x05_Counter_Clockwise
Connections:
- net +3.3V: now also J11.1 (Pin_1), J11.2 (Pin_2), J11.3 (Pin_3), J11.4 (Pin_4), J11.5 (Pin_5)
- net GND: now also J11.10 (Pin_10), J11.6 (Pin_6), J11.7 (Pin_7), J11.8 (Pin_8), J11.9 (Pin_9)
- net MIC_IO: now also U10.20 (PA4); no longer U10.53 (PC12)
- net UI_LED_R: now also U10.53 (PC12); no longer U10.20 (PA4)

Commit message: Final Version of EV14
Parts:
- removed J10: Conn_02x05_Counter_Clockwise, Hactar_Footprints:HDR-SMD_10P-P2.54-V-F-R2-C5-LS7.1-1, symbol Connector_Generic:Conn_02x05_Counter_Clockwise
- removed J4: AudioJack4, Hactar_Footprints:AUDIO-SMD_PJ-242, symbol Connector_Audio:AudioJack4
- removed R37: 100k, Resistor_SMD:R_0402_1005Metric, symbol Device:R_US
- removed R63: 1k0, Resistor_SMD:R_0402_1005Metric, symbol Device:R_US
- added C49: 100n, Capacitor_SMD:C_0402_1005Metric, symbol Device:C
- added CN2: PJ-242, Hactar_Footprints:AUDIO-SMD_PJ-242D-SMT, symbol Hactar_Symbols:PJ-242
- added J10: Conn_02x04_Odd_Even, Hactar_Footprints:HDR-SMD_8P-P2.54-V-M-R2-C4-LS7.4, symbol Connector_Generic:Conn_02x04_Odd_Even
- added R75: 4k7, Resistor_SMD:R_0402_1005Metric, symbol Device:R_US
Connections:
- net +3.3V: now also R75.2
- net GND: now also C49.2
- net GNDA: now also CN2.4
- net MGMT_BOOT: now also J10.8 (Pin_8)
- net MGMT_NRST: now also J10.6 (Pin_6)
- net MGMT_SWCLK: now also J10.2 (Pin_2)
- net MGMT_SWDIO: now also J10.4 (Pin_4)
- net MIC_IO: now also C49.1
- net MIC_N: now also CN2.2
- net NET_BOOT: now also J10.1 (Pin_1)
- net NET_NRST: now also J10.7 (Pin_7)
- net NET_RX1_MGMT: now also J10.5 (Pin_5)
- net NET_TX1_MGMT: now also J10.3 (Pin_3)
- net at Q2.2 (G), Q2.5 (G), Q3.2 (G): now also CN2.5, R75.1
- net at Q2.3 (D): now also CN2.6
- net UI_SCL renamed UI_SCL1
- net UI_SDA renamed UI_SDA1
Other:
- note added: "EV14 layer build up: top: High Speed second: GND third: 3.3V bottom: Low Speed"
- note removed: "EV13 layer build up: top: High Speed second: GND third: 3.3V bottom: Low Speed"
- moved on the sheet: J11
