File: hardware/ev15/ev15.kicad_sch (KiCad schematic)
At the start: 165 parts, among them CN1 Conn_05x02_Female, CN2 PJ-242, J1 USB_C_Receptacle, J10 Conn_02x04_Odd_Even, J11 Conn_02x05_Counter_Clockwise, J2 Conn_01x02_Socket, J3 AudioJack4, J4 Conn_01x18_MountingPin, J5 Conn_02x03_Odd_Even, J7 Conn_02x05_Counter_Clockwise, J8 Conn_02x05_Counter_Clockwise, J9 Conn_02x05_Counter_Clockwise, Q1 2N7002, SW1 SW_SPDT, SW2 SW_Push, SW3 SW_Push, SW4 SW_Push, SW5 SW_Push, U1 BQ21040DBV, U10 STM32F405RGTx, U2 USBLC6-2P6, U3 STM32F072CBTx, U4 CH340C, U5 TPS63060, U6 WM8960CGEFL/RV, U7 ESP32-S3-WROOM-1, U8 M24C02-RMN6TP, U9 BM14B(0.8)-24DS-0.4V(53), Y1 Crystal_GND24

Commit message: chore: renamed ev14a to ev15
Other:
- title: EV14 FINN BERG & BRETT REGNIER -> EV15 FINN BERG & BRETT REGNIER
Changed lines of the file:
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@@
 	(paper "A2")
 	(title_block
-		(title "EV14 FINN BERG & BRETT REGNIER")
+		(title "EV15 FINN BERG & BRETT REGNIER")
 		(date "2025-07-25")
+		(rev "EV15")
 		(company "CISCO SYSTEMS INC")
 	)

Commit message: feat: update kb connector part number to one with more stock
Parts:
- U9: JLCPCB Part # C9900001863 -> C3640874
Changed lines of the file:
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@@
 			)
 		)
-		(property "JLCPCB Part #" "C9900001863"
+		(property "JLCPCB Part #" "C3640874"
 			(at 304.8 363.22 0)
 			(effects
