File: hardware/ev19/ui.kicad_sch (KiCad schematic)
At the start: 43 parts, among them CN3 BM14B(0.8)-24DS-0.4V(53), J14 Conn_01x18_MountingPin, Q5 2N7002, SW4 SW_Push, SW5 SW_Push, SW6 SW_Push, SW7 SW_Push, U10 STM32F405RGTx

Commit message: Added missing footprints, used kicad10 wizard tool to design them, designed starting point of the board layout
Parts:
- J14: footprint (none) -> Connector_FFC-FPC:Hirose_FH12-18S-0.5SH_1x18-1MP_P0.50mm_Horizontal; JLCPCB Part # (none) -> C2856802
Changed lines of the file:
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@@
 			)
 		)
-		(property "Footprint" ""
+		(property "Footprint" "Connector_FFC-FPC:Hirose_FH12-18S-0.5SH_1x18-1MP_P0.50mm_Horizontal"
 			(at 250.19 137.16 0)
 			(hide yes)
@@
 			(at 250.19 137.16 0)
 			(hide yes)
+			(show_name no)
+			(do_not_autoplace no)
+			(effects
+				(font
+					(size 1.27 1.27)
+				)
+			)
+		)
+		(property "JLCPCB Part #" "C2856802"
+			(at 250.19 137.16 0)
+			(hide yes)
