File: hardware/ev19/ui.kicad_sch (KiCad schematic)
At the start: 43 parts, among them CN3 BM14B(0.8)-24DS-0.4V(53), J13 Conn_01x08_Pin, Q5 2N7002, SW4 SW_Push, SW5 SW_Push, SW6 SW_Push, SW7 SW_Push, U10 STM32F405RGTx

Commit message: Redesigned digital section again to fit the battery better. Chose where the screen connector and battery connector go
Parts:
- removed J13: Conn_01x08_Pin, Connector_PinHeader_2.54mm:PinHeader_1x08_P2.54mm_Vertical_SMD_Pin1Left, symbol Connector:Conn_01x08_Pin
- added J14: Diplay_Connector, Connector_JST:JST_PH_S8B-PH-SM4-TB_1x08-1MP_P2.00mm_Horizontal, symbol Connector_Generic_MountingPin:Conn_01x08_MountingPin
- SW4, SW5: footprint Hactar_Footprints:SW-SMD_4P-L5.1-W5.1-P3.70-LS6.5-TL_H1.5 -> Hactar_Footprints:SW-SMD_SHOU_TS36CA-0.6; symbol Hactar_Symbols:SW4_Push -> Switch:SW_Push; JLCPCB Part # C318886 -> C2906288
Connections:
- net +3.3V: now also J14.8 (Pin_8); no longer SW4.2, SW5.2
- net DISP_BL: now also J14.1 (Pin_1)
- net DISP_CS: now also J14.4 (Pin_4)
- net DISP_DC: now also J14.3 (Pin_3)
- net DISP_RST: now also J14.2 (Pin_2)
- net GND: now also J14.7 (Pin_7)
- net SPI1_CLK: now also J14.5 (Pin_5)
- net SPI1_MOSI: now also J14.6 (Pin_6)
- net at C47.1, R58.2, R62.2: now also SW5.2; no longer SW5.3, SW5.4
- net at C46.1, R57.2, R61.2: now also SW4.2; no longer SW4.3, SW4.4
- no-connect marks 2 -> 3
Changed lines of the file:
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@@
 	)
 	(no_connect
+		(at 251.46 102.87)
+	)
+	(no_connect
 		(at 245.11 40.64)
 	)
@@
 	)
 	(symbol
-		(lib_id "Hactar_Symbols:SW4_Push")
+		(lib_id "Switch:SW_Push")
 		(at 185.42 102.87 0)
 		(unit 1)
@@
 			)
 		)
-		(property "Footprint" "Hactar_Footprints:SW-SMD_4P-L5.1-W5.1-P3.70-LS6.5-TL_H1.5"
-			(at 185.42 102.87 0)
+		(property "Footprint" "Hactar_Footprints:SW-SMD_SHOU_TS36CA-0.6"
+			(at 185.42 97.79 0)
 			(hide yes)
 			(show_name no)
@@
 		)
 		(property "Datasheet" ""
-			(at 185.42 102.87 0)
+			(at 185.42 97.79 0)
 			(hide yes)
 			(show_name no)
@@
 			)
 		)
-		(property "JLCPCB Part #" "C318886"
+		(property "JLCPCB Part #" "C2906288"
 			(at 180.848 100.584 0)
 			(hide yes)
@@
 		(pin "2"
 		)
-		(pin "3"
-		)
-		(pin "4"
-		)
 		(instances
 			(project "ev19"
@@
 	)
 	(symbol
+		(lib_id "Connector_Generic_MountingPin:Conn_01x08_MountingPin")
+		(at 251.46 118.11 0)
+		(mirror x)
+		(unit 1)
+		(body_style 1)
+		(exclude_from_sim no)
+		(in_bom yes)
+		(on_board yes)
+		(in_pos_files yes)
+		(dnp no)
+		(property "Reference" "J14"
+			(at 231.648 127 0)
+			(show_name no)
+			(do_not_autoplace no)
+			(effects
+				(font
+					(size 1.27 1.27)
+				)
+				(justify left)
+			)
+		)
+		(property "Value" "Diplay_Connector"
+			(at 230.632 129.794 0)
+			(show_name no)
+			(do_not_autoplace no)
+			(effects
+				(font
+					(size 1.27 1.27)
+				)
+				(justify left)
+			)
+		)
+		(property "Footprint" "Connector_JST:JST_PH_S8B-PH-SM4-TB_1x08-1MP_P2.00mm_Horizontal"
+			(at 251.46 118.11 0)
+			(hide yes)
+			(show_name no)
+			(do_not_autoplace no)
+			(effects
+				(font
+					(size 1.27 1.27)
+				)
+			)
+		)
+		(property "Datasheet" ""
+			(at 251.46 118.11 0)
+			(hide yes)
+			(show_name no)
+			(do_not_autoplace no)
+			(effects
+				(font
+					(size 1.27 1.27)
+				)
+			)
+		)
+		(property "Description" "Generic connectable mounting pin connector, single row, 01x08, script generated (kicad-library-utils/schlib/autogen/connector/)"
+			(at 251.46 118.11 0)
+			(hide yes)
+			(show_name no)
+			(do_not_autoplace no)
+			(effects
+				(font
+					(size 1.27 1.27)
+				)
+			)
+		)
+		(property "JLCPCB Part #" "C265121"
+			(at 251.46 118.11 0)
+			(hide yes)
+			(show_name no)
+			(do_not_autoplace no)
+			(effects
+				(font
+					(size 1.27 1.27)
+				)
+			)
+		)
+		(pin "5"
+		)
+		(pin "8"
+		)
+		(pin "MP"
+		)
+		(pin "4"
+		)
+		(pin "1"
+		)
+		(pin "6"
+		)
+		(pin "3"
+		)
+		(pin "2"
+		)
+		(pin "7"
+		)
+		(instances
+			(project "ev19"
+				(path "/bd865368-262b-4f76-b7a6-1673c2cb0f8c/3dc257c8-f72f-473f-bf23-b8869158b2ba"
+					(reference "J14")
+					(unit 1)
+				)
+			)
+		)
+	)
+	(symbol
 		(lib_id "Device:R_US")
 		(at 194.31 107.95 180)
@@
 	)
 	(symbol
-		(lib_id "Hactar_Symbols:SW4_Push")
+		(lib_id "Switch:SW_Push")
 		(at 186.69 72.39 0)
 		(unit 1)
@@
 			)
 		)
-		(property "Footprint" "Hactar_Footprints:SW-SMD_4P-L5.1-W5.1-P3.70-LS6.5-TL_H1.5"
-			(at 186.69 72.39 0)
+		(property "Footprint" "Hactar_Footprints:SW-SMD_SHOU_TS36CA-0.6"
+			(at 186.69 67.31 0)
 			(hide yes)
 			(show_name no)
@@
 		)
 		(property "Datasheet" ""
-			(at 186.69 72.39 0)
+			(at 186.69 67.31 0)
 			(hide yes)
 			(show_name no)
@@
 			)
 		)
-		(property "JLCPCB Part #" "C318886"
+		(property "JLCPCB Part #" "C2906288"
 			(at 182.118 70.104 0)
 			(hide yes)
@@
 		(pin "2"
 		)
-		(pin "4"
-		)
-		(pin "3"
-		)
 		(instances
 			(project "ev19"
@@
 					(unit 1)
 				)
-			)
-		)
-	)
-	(symbol
-		(lib_id "Connector:Conn_01x08_Pin")
-		(at 251.46 118.11 180)
-		(unit 1)
-		(body_style 1)
-		(exclude_from_sim no)
-		(in_bom yes)
-		(on_board yes)
-		(in_pos_files yes)
-		(dnp no)
-		(property "Reference" "J13"
-			(at 237.744 105.664 0)
-			(show_name no)
-			(do_not_autoplace no)
-			(effects
-				(font
-					(size 1.27 1.27)
-				)
-				(justify right)
-			)
-		)
-		(property "Value" "Conn_01x08_Pin"
-			(at 237.49 103.378 0)
-			(show_name no)
-			(do_not_autoplace no)
-			(effects
-				(font
-					(size 1.27 1.27)
-				)
-				(justify right)
-			)
-		)
-		(property "Footprint" "Connector_PinHeader_2.54mm:PinHeader_1x08_P2.54mm_Vertical_SMD_Pin1Left"
-			(at 251.46 118.11 0)
-			(hide yes)
-			(show_name no)
-			(do_not_autoplace no)
-			(effects
-				(font
-					(size 1.27 1.27)
-				)
-			)
-		)
-		(property "Datasheet" ""
-			(at 251.46 118.11 0)
-			(hide yes)
-			(show_name no)
-			(do_not_autoplace no)
-			(effects
-				(font
-					(size 1.27 1.27)
-				)
-			)
-		)
-		(property "Description" "Generic connector, single row, 01x08, script generated"
-			(at 251.46 118.11 0)
-			(hide yes)
-			(show_name no)
-			(do_not_autoplace no)
-			(effects
-				(font
-					(size 1.27 1.27)
-				)
-			)
-		)
-		(pin "3"
-		)
-		(pin "5"
-		)
-		(pin "2"
-		)
-		(pin "4"
-		)
-		(pin "1"
-		)
-		(pin "6"
-		)
-		(pin "7"
-		)
-		(pin "8"
-		)
-		(instances
-			(project "ev19"
-				(path "/bd865368-262b-4f76-b7a6-1673c2cb0f8c/3dc257c8-f72f-473f-bf23-b8869158b2ba"
-					(reference "J13")
-					(unit 1)
-				)

Commit message: Moved debug connector so it wasnt in the way of ht screen connector beging plugged in
Changed lines of the file:
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@@
 	(wire
 		(pts
-			(xy 128.27 62.23) (xy 148.59 62.23)
+			(xy 128.27 62.23) (xy 143.51 62.23)
 		)
 		(stroke
@@
 	(wire
 		(pts
-			(xy 148.59 105.41) (xy 128.27 105.41)
+			(xy 143.51 105.41) (xy 128.27 105.41)
 		)
 		(stroke
@@
 	)
 	(label "VOLUME-"
-		(at 148.59 62.23 180)
+		(at 143.51 62.23 180)
 		(effects
 			(font
@@
 	)
 	(label "KB_COL5"
-		(at 148.59 105.41 180)
+		(at 143.51 105.41 180)
 		(effects
 			(font
@@
 		)
 	)
+	(global_label "VOLUME-"
+		(shape input)
+		(at 143.51 62.23 0)
+		(fields_autoplaced yes)
+		(effects
+			(font
+				(size 1.27 1.27)
+			)
+			(justify left)
+		)
+		(property "Intersheetrefs" "${INTERSHEET_REFS}"
+			(at 155.4457 62.23 0)
+			(hide yes)
+			(show_name no)
+			(do_not_autoplace no)
+			(effects
+				(font
+					(size 1.27 1.27)
+				)
+				(justify left)
+			)
+		)
+	)
+	(global_label "KB_COL5"
+		(shape input)
+		(at 143.51 105.41 0)
+		(fields_autoplaced yes)
+		(effects
+			(font
+				(size 1.27 1.27)
+			)
+			(justify left)
+		)
+		(property "Intersheetrefs" "${INTERSHEET_REFS}"
+			(at 154.8409 105.41 0)
+			(hide yes)
+			(show_name no)
+			(do_not_autoplace no)
+			(effects
+				(font
+					(size 1.27 1.27)
+				)
+				(justify left)
+			)
+		)
+	)

Commit message: Almost done layout out all of the traces
Connections:
- net KB_COL5 renamed UI_DEBUG_1
- net VOLUME- renamed UI_DEBUG_2
Changed lines of the file:
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@@
 	(wire
 		(pts
-			(xy 128.27 62.23) (xy 143.51 62.23)
+			(xy 128.27 62.23) (xy 139.7 62.23)
 		)
 		(stroke
@@
 	(wire
 		(pts
-			(xy 143.51 105.41) (xy 128.27 105.41)
+			(xy 138.43 105.41) (xy 128.27 105.41)
 		)
 		(stroke
@@
 	)
 	(label "VOLUME-"
-		(at 143.51 62.23 180)
+		(at 139.7 62.23 180)
 		(effects
 			(font
@@
 	)
 	(label "KB_COL5"
-		(at 143.51 105.41 180)
+		(at 138.43 105.41 180)
 		(effects
 			(font
@@
 		)
 	)
-	(global_label "VOLUME-"
+	(global_label "UI_DEBUG_2"
 		(shape input)
-		(at 143.51 62.23 0)
+		(at 139.7 62.23 0)
 		(fields_autoplaced yes)
 		(effects
@@
 		)
 		(property "Intersheetrefs" "${INTERSHEET_REFS}"
-			(at 155.4457 62.23 0)
+			(at 154.0547 62.23 0)
 			(hide yes)
 			(show_name no)
@@
 		)
 	)
-	(global_label "KB_COL5"
+	(global_label "UI_DEBUG_1"
 		(shape input)
-		(at 143.51 105.41 0)
+		(at 138.43 105.41 0)
 		(fields_autoplaced yes)
 		(effects
@@
 		)
 		(property "Intersheetrefs" "${INTERSHEET_REFS}"
-			(at 154.8409 105.41 0)
+			(at 152.7847 105.41 0)
 			(hide yes)
 			(show_name no)

Commit message: Updated schematic and pcb to output a file jlcpcb expects
Parts:
- J14: FT Rotation Offset (none) -> 180
Other:
- company: (none) -> CISCO SYSTEMS INC
- title: (none) -> HACTAR - Finn Berg & Brett Regnier
Changed lines of the file:
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@@
 	(generator_version "10.0")
 	(paper "A4")
+	(title_block
+		(title "HACTAR - Finn Berg & Brett Regnier")
+		(date "2026-07-27")
+		(rev "EV19")
+		(company "CISCO SYSTEMS INC")
+	)
 	(rectangle
 		(start 173.99 20.32)
@@
 			(at 251.46 118.11 0)
 			(hide yes)
+			(show_name no)
+			(do_not_autoplace no)
+			(effects
+				(font
+					(size 1.27 1.27)
+				)
+			)
+		)
+		(property "FT Rotation Offset" "180"
+			(at 251.46 118.11 0)
+			(hide yes)
