File: hardware/ev19/ev19.kicad_sch (KiCad schematic)
At the start: 156 parts, among them CN1 Conn_05x02_Female, J1 USB_C_Receptacle, J10 USB_C_Receptacle, J11 Conn_02x05_Counter_Clockwise, J2 BATT_CONN, J4 Conn_02x03_Odd_Even, J5 Conn_02x03_Odd_Even, J6 Conn_02x05_Counter_Clockwise, J7 Conn_02x05_Counter_Clockwise, J8 Conn_02x05_Counter_Clockwise, J9 Conn_02x05_Counter_Clockwise, Q1 2N7002, Q2 2N7002, Q3 2N7002, Q4 2N7002, SW1 SW_SPDT, SW2 SW_Push, SW3 SW_Push, U1 BQ21040DBV, U12 XC6227C301MR-G, U2 USBLC6-2P6, U3 STM32F072CBTx, U4 CH340C, U5 TPS63060, U7 ESP32-S3-WROOM-1, U9 TPS2116DRL, Y1 Crystal_GND24

Commit message: Changed debug ports to 32pin female headers, laid out more of the digital section, drew square where screen should sit
Parts:
- removed J6, J7, J8, J9: Conn_02x05_Counter_Clockwise, Hactar_Footprints:HDR-SMD_10P-P2.54-V-F-R2-C5-LS7.1-1, symbol Connector_Generic:Conn_02x05_Counter_Clockwise
- removed R66, R67, R68, R69: 4k7, Resistor_SMD:R_0402_1005Metric, symbol Device:R_US
- removed R70, R71, R72, R73, R74: 1k0, Resistor_SMD:R_0402_1005Metric, symbol Device:R_US
- added J13, J15: Conn_02x16_Counter_Clockwise, Connector_PinHeader_2.54mm:PinHeader_2x16_P2.54mm_Vertical_SMD, symbol Connector_Generic:Conn_02x16_Counter_Clockwise
- added R66, R67, R68, R69: 4k7, Resistor_SMD:R_0402_1005Metric, symbol Device:R_Small_US
- added R70, R71, R73, R74: 1k0, Resistor_SMD:R_0402_1005Metric, symbol Device:R_Small_US
Connections:
- net GND: now also J13.17 (Pin_17), J13.18 (Pin_18), J13.19 (Pin_19), J13.20 (Pin_20), J13.21 (Pin_21), J13.22 (Pin_22), J13.23 (Pin_23), J13.24 (Pin_24), J13.25 (Pin_25), J13.26 (Pin_26), J13.27 (Pin_27), J13.28 (Pin_28), J13.29 (Pin_29), J13.30 (Pin_30), J13.31 (Pin_31), J13.32 (Pin_32), J15.17 (Pin_17), J15.18 (Pin_18), J15.19 (Pin_19), J15.20 (Pin_20), J15.21 (Pin_21), J15.22 (Pin_22), J15.23 (Pin_23), J15.24 (Pin_24), J15.25 (Pin_25), J15.26 (Pin_26), J15.27 (Pin_27), J15.28 (Pin_28), J15.29 (Pin_29), J15.30 (Pin_30), J15.31 (Pin_31), J15.32 (Pin_32), R66.2, R67.2, R68.2, R69.2
- net I2S_ADCDAT: now also J15.8 (Pin_8), R69.1
- net I2S_BCLK: now also J15.9 (Pin_9), R68.1
- net I2S_DACDAT: now also J15.7 (Pin_7), R67.1
- net I2S_DACLRC: now also J15.10 (Pin_10), R66.1
- net KB_COL5: now also R74.2
- net MCLK: now also J15.1 (Pin_1)
- net MGMT_DEBUG_1: now also J15.12 (Pin_12)
- net MGMT_DEBUG_2: now also J15.11 (Pin_11)
- net NET_BOOT: now also J13.7 (Pin_7)
- net NET_DEBUG_1: now also R70.1
- net NET_DEBUG_2: now also R71.1
- net NET_NRST: now also J13.8 (Pin_8)
- net NET_RX1_MGMT: now also J13.6 (Pin_6)
- net NET_TX1_MGMT: now also J13.5 (Pin_5)
- net SPI1_CLK: now also J15.3 (Pin_3)
- net SPI1_MISO: now also J15.4 (Pin_4)
- net SPI1_MOSI: now also J15.2 (Pin_2)
- net UI_BOOT0: now also J13.12 (Pin_12)
- net UI_CTS2_NET: now also J13.16 (Pin_16)
- net UI_NRST: now also J13.11 (Pin_11)
- net UI_RTS2_NET: now also J13.15 (Pin_15)
- net UI_RX1_MGMT: now also J13.10 (Pin_10)
- net UI_RX2_NET: now also J13.14 (Pin_14)
- net UI_SCL1: now also J15.6 (Pin_6)
- net UI_SDA1: now also J15.5 (Pin_5)
- net UI_TX1_MGMT: now also J13.9 (Pin_9)
- net UI_TX2_NET: now also J13.13 (Pin_13)
- net USB_RX1_MGMT: now also J13.2 (Pin_2)
- net USB_TX1_MGMT: now also J13.1 (Pin_1)
- net VOLUME-: now also R73.2
- net USB_DTR renamed USB_DTR_MGMT
- net USB_DTR_MGMT: now also J13.4 (Pin_4)
- net USB_RTS renamed USB_RTS_MGMT
- net USB_RTS_MGMT: now also J13.3 (Pin_3)
- new net: J15.14 (Pin_14), R73.1
- new net: J15.13 (Pin_13), R74.1
- new net: J15.16 (Pin_16), R71.2
- new net: J15.15 (Pin_15), R70.2
- no-connect marks 42 -> 39
Other:
- note removed: "GPIO DEBUG"
- note removed: "I2S + I2C DEBUG"
- note removed: "NET SERIAL UPLOADER + SPI"
- note removed: "SERIAL DEBUG"
- moved on the sheet: J10, J11

Commit message: Forgot to push the schematic
Parts:
- added H5: MountingHole, MountingHole:MountingHole_2.7mm_M2.5, symbol Mechanical:MountingHole
Changed lines of the file:
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@@
 	(rectangle
 		(start 153.67 222.25)
-		(end 180.34 247.65)
+		(end 180.34 255.27)
 		(stroke
 			(width 0)
@@
 					(unit 1)
 				)
+			)
+		)
+	)
+	(symbol
+		(lib_id "Mechanical:MountingHole")
+		(at 158.75 247.65 0)
+		(unit 1)
+		(body_style 1)
+		(exclude_from_sim no)
+		(in_bom no)
+		(on_board yes)
+		(in_pos_files yes)
+		(dnp no)
+		(fields_autoplaced yes)
+		(property "Reference" "H5"
+			(at 161.29 246.3799 0)
+			(show_name no)
+			(do_not_autoplace no)
+			(effects
+				(font
+					(size 1.27 1.27)
+				)
+				(justify left)
+			)
+		)
+		(property "Value" "MountingHole"
+			(at 161.29 248.9199 0)
+			(show_name no)
+			(do_not_autoplace no)
+			(effects
+				(font
+					(size 1.27 1.27)
+				)
+				(justify left)
+			)
+		)
+		(property "Footprint" "MountingHole:MountingHole_2.7mm_M2.5"
+			(at 158.75 247.65 0)
+			(hide yes)
+			(show_name no)
+			(do_not_autoplace no)
+			(effects
+				(font
+					(size 1.27 1.27)
+				)
+			)
+		)
+		(property "Datasheet" ""
+			(at 158.75 247.65 0)
+			(hide yes)
+			(show_name no)
+			(do_not_autoplace no)
+			(effects
+				(font
+					(size 1.27 1.27)
+				)
+			)
+		)
+		(property "Description" "Mounting Hole without connection"
+			(at 158.75 247.65 0)
+			(hide yes)
+			(show_name no)
+			(do_not_autoplace no)
+			(effects
+				(font
+					(size 1.27 1.27)
+				)
+			)
+		)
+		(property "JLCPCB Position Offset" ""
+			(at 158.75 247.65 0)
+			(hide yes)
+			(show_name no)
+			(do_not_autoplace no)
+			(effects
+				(font
+					(size 1.27 1.27)
+				)
+			)
+		)
+		(property "Sim.Type" ""
+			(at 158.75 247.65 0)
+			(hide yes)
+			(show_name no)
+			(do_not_autoplace no)
+			(effects
+				(font
+					(size 1.27 1.27)
+				)
+			)
+		)
+		(instances
+			(project "ev19"
+				(path "/bd865368-262b-4f76-b7a6-1673c2cb0f8c"
+					(reference "H5")
+					(unit 1)
+				)
