File: hardware/ev19/eeprom.kicad_sch (KiCad schematic)
At the start: 2 parts, among them U8 M24C02-RMN6TP

Commit message: Almost done layout out all of the traces
Parts:
- U8: value M24C02-RMN6TP -> M24C02-RDW6TP; footprint Package_SO:SOIC-8_3.9x4.9mm_P1.27mm -> Package_SO:TSSOP-8_3x3mm_P0.65mm; JLCPCB Part # C83836 -> C152731
Changed lines of the file:
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@@
 			)
 		)
-		(property "Value" "M24C02-RMN6TP"
+		(property "Value" "M24C02-RDW6TP"
 			(at 60.706 59.182 0)
 			(show_name no)
@@
 			)
 		)
-		(property "Footprint" "Package_SO:SOIC-8_3.9x4.9mm_P1.27mm"
+		(property "Footprint" "Package_SO:TSSOP-8_3x3mm_P0.65mm"
 			(at 60.96 40.64 0)
 			(hide yes)
@@
 			)
 		)
-		(property "JLCPCB Part #" "C83836"
+		(property "JLCPCB Part #" "C152731"
 			(at 60.96 49.53 0)
 			(hide yes)

Commit message: Updated schematic and pcb to output a file jlcpcb expects
Other:
- title: EEPROM -> HACTAR - Finn Berg & Brett Regnier
Changed lines of the file:
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@@
 	(paper "A4")
 	(title_block
-		(title "EEPROM")
-		(date "2026-06-18")
+		(title "HACTAR - Finn Berg & Brett Regnier")
+		(date "2026-07-27")
 		(rev "EV19")
 		(company "CISCO SYSTEMS INC")

Commit message: Fixed eeprom footprint, moved mount holes, added ptt buttons, adjusted location of screen jst connector
Parts:
- U8: footprint Package_SO:TSSOP-8_3x3mm_P0.65mm -> Package_SO:TSSOP-8_4.4x3mm_P0.65mm
Changed lines of the file:
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@@
 			)
 		)
-		(property "Footprint" "Package_SO:TSSOP-8_3x3mm_P0.65mm"
+		(property "Footprint" "Package_SO:TSSOP-8_4.4x3mm_P0.65mm"
 			(at 60.96 40.64 0)
 			(hide yes)
